File: Schematic/I&O_Epander/I&O_Epander.sch (KiCad schematic (older format))
At the start: 70 parts, among them J1 RJ45-Unshielded, J10 RJ45-Unshielded, J11 RJ45-Unshielded, J12 KLDVHCX-0202-A, J13 RJ45-Unshielded, J14 RJ45-Unshielded, J2 RJ45-Unshielded, J3 RJ45-Unshielded, J4 RJ45-Unshielded, J5 RJ45-Unshielded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

Commit message: KiCAD upgrade
Upgrade schematic and pcb files for KiCad v5.
Make 8-pin dip holes larger for crimped-pin sockets
InteractiveBOM plugin v1.1 board stuffing files generated.
Parts:
- C1, C10, C12, C14, C15, C17, C2, C3, C4, C5, C6, C7, C8, C9: symbol CAP_NP -> NewUnsorted:CAP_NP
- C11, C13, C16, C18: symbol CAP_P -> NewUnsorted:CAP_P
- J1, J10, J11, J13, J14, J2, J3, J4, J5, J6, J7, J8: symbol RJ45-Unshielded -> NewUnsorted:RJ45-Unshielded
- J12, J9: symbol JACK-PWR -> NewUnsorted:JACK-PWR
- MH1: symbol MOUNTING_HOLE_PTH -> NewUnsorted:MOUNTING_HOLE_PTH
- MH2, MH3, MH4: symbol MOUNTING_HOLE_NPTH -> NewUnsorted:MOUNTING_HOLE_NPTH
- Q1: symbol Q_NMOS_SGD -> NewUnsorted:Q_NMOS_SGD
- R1, R10, R11, R12, R13, R2, R3, R4, R5, R6, R7, R8, R9: symbol RES -> NewUnsorted:RES
- U1: symbol 74HC595 -> NewUnsorted:74HC595
- U10, U8: symbol DS8921 -> NewUnsorted:DS8921
- U2: symbol 74HC165 -> NewUnsorted:74HC165
- U3, U4, U5, U6: symbol 75C1168 -> NewUnsorted:75C1168
- U7: symbol uA9637AC -> NewUnsorted:uA9637AC
- U9: symbol uA9638C -> NewUnsorted:uA9638C
- XU1, XU2, XU3, XU4, XU5, XU6: symbol IC_Socket16 -> NewUnsorted:IC_Socket16
- XU10, XU7, XU8, XU9: symbol IC_Socket08 -> NewUnsorted:IC_Socket08
Connections:
- wire segments 330 -> 430
Other:
- moved on the sheet: R2, R3, R4, R5
