File: Schematic/Logic&Oscillator/Logic&Oscillator.sch (KiCad schematic (older format))
At the start: 33 parts, among them J1 KLDVHCX-0202-A, J2 KLDVHCX-0202-A, J3 RJ45-Unshielded, J4 RJ45-Unshielded, Q1 VN3205, U1 ICM7555, U2 ARDUINO_Pro-Mini 5v, U3 uA9638C, U4 uA9638C, U5 DS8921

Commit message: KiCAD upgrade
Upgrade schematic and pcb files for KiCad v5.
Make 8-pin dip holes larger for crimped-pin sockets
InteractiveBOM plugin v1.1 board stuffing files generated.
Parts:
- C1, C10, C11, C2, C4, C5, C7, C9: symbol CAP_NP -> NewUnsorted:CAP_NP
- C3, C6, C8: symbol CAP_P -> NewUnsorted:CAP_P
- J1, J2: symbol JACK-PWR -> NewUnsorted:JACK-PWR
- J3, J4: symbol RJ45-Unshielded -> NewUnsorted:RJ45-Unshielded
- MH1: symbol MOUNTING_HOLE_PTH -> NewUnsorted:MOUNTING_HOLE_PTH
- MH2, MH3, MH4: symbol MOUNTING_HOLE_NPTH -> NewUnsorted:MOUNTING_HOLE_NPTH
- Q1: symbol Q_NMOS_SGD -> NewUnsorted:Q_NMOS_SGD
- R1, R3, R4: symbol RES -> NewUnsorted:RES
- R2: symbol POT_W2 -> NewUnsorted:POT_W2
- U1: symbol ICM7555 -> NewUnsorted:ICM7555
- U2: symbol ARDUINO_Pro-Mini -> Arduino:ARDUINO_Pro-Mini
- U3, U4: symbol uA9638C -> NewUnsorted:uA9638C
- U5: symbol DS8921 -> NewUnsorted:DS8921
- XU1, XU3, XU4, XU5: symbol IC_Socket08 -> NewUnsorted:IC_Socket08
Connections:
- wire segments 112 -> 145
